File: BenchTopPowerSupply.sch (EAGLE design)
At the start: 129 parts, among them U10 E2A-T220-25E, U7 STM32F103C8T6, U8 E2A-T220-25E, U9 E2A-T220-25E, X1 5566-24, Y1 8MHZ

Commit message: Fixing schematic issues
Parts:
- added R34: 1M, rcl:R-EU_R1206
Connections:
- new net N$10: C18.2, C19.2
- net BOOT1: now also U7.PB2; no longer U7.PB1
- net GND: no longer C18.2, C19.2
- net N$3: now also R34.2
- net N$5: now also R34.1
Other:
- moved on the sheet: BOOT, C13, C14, C15, C16, C17, C18, C19, C20, C23, I2C, LED1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

Commit message: Adding mounting holes to the design and experimenting with JLCPCB SMT assembly
Parts:
- removed PS_FAN: (no value), pinhead:PINHD-1X2
- added 3V3_PWR, 5V_PWR: PINHD-2X3, Connector:PINHD-2X3
- added C34: 100nF, rcl:C-EUC1206
- added C35, C37: 100nF, rcl:CPOL-EUE5-5
- added C36, C38: 100uF, rcl:C-EUC1206
- added D4, D5: 1N4148DO35-7, diode:1N4148DO35-7
- added IN_FAN, OUT_FAN: 61300211121, Headers:61300211121
- added Q1: NPN, Transistor:NPN_TO92
- added Q2, Q3: IRF510, transistor-power:IRF512
- added R35, R36, R37, R40: 10k, rcl:R-EU_R1206
- added R38, R39: 470, rcl:R-EU_R1206
- added SPI: PINHD-1X3, Connector:PINHD-1X3
- R1: value (none) -> 100K
Connections:
- new net IN_FAN_PWM: D4.C, R38.2, U7.PB10
- new net N$26: Q1.B, R35.2
- new net N$30: D4.A, Q2.G, R37.2, R38.1
- new net N$31: IN_FAN.1, Q2.D
- new net N$32: D5.A, Q3.G, R39.1, R40.2
- new net N$35: OUT_FAN.1, Q3.D
- new net OUT_FAN_PWM: D5.C, R39.2, U7.PB11
- new net SPI_MISO: SPI.2, U7.PB4
- new net SPI_MOSI: SPI.3, U7.PB5
- new net SPI_NSS: U7.PA15
- new net SPI_SCK: SPI.1, U7.PB3
- new net TEMP_SENS: R35.1, R36.2, U7.PB0
- net +12V: now also C34.1, IN_FAN.2, OUT_FAN.2, Q1.E; no longer PS_FAN.1
- net +3V3: now also 3V3_PWR.1, 3V3_PWR.3, 3V3_PWR.5, C35.+, C36.2
- net +5V: now also 5V_PWR.1, 5V_PWR.3, 5V_PWR.5, C37.+, C38.2
- net GND: now also 3V3_PWR.2, 3V3_PWR.4, 3V3_PWR.6, 5V_PWR.2, 5V_PWR.4, 5V_PWR.6, C34.2, C35.-, C36.1, C37.-, C38.1, Q1.C, Q2.S, Q3.S, R36.1, R37.1, R40.1; no longer PS_FAN.2
Other:
- note added: "100KOhm"
- note added: "IRF510"
- note added: "LM35 Module"
- note removed: "Screw Terminals need replaced cant access them from layout"
- moved on the sheet: I2C, R24, R25, UART

Commit message: Changing to surface mount inductors, reduce noise on board, hopefully. Will need to redo layout however and figure out how to solder them
Parts:
- L1, L2, L3: value A26GFC -> DR125; device inductors:A26GFC -> inductors:DR125
- R1: value 100K -> 100k
Other:
- note added: "CHECK INDUCTOR PART AND CAP PART NEED TO REDO LAYOUT FOR INDUCTORS 3D CAD MODEL FOR INDUCTORS TOO"
- note removed: "CHECK INDUCTOR PART AND CAP PART"
